File: Arm Motor PCBs J4/Hardware/ArmMotorPCBJ4/ArmMotorPCBJ4.kicad_pcb (KiCad board)
At the start: 2 copper layers, 35.6 x 45.7 mm, 5 parts

Commit message: gerbs added and zipped
Other:
- board text added: "ARM MOTOR PCB J4 2022"
- board text removed: "Motor PCB Breakout J4 2022"
