File: NO_Breakout_Board/NO_Breakout_Board.kicad_pcb (KiCad board)
At the start: 2 copper layers, 29.7 x 15.5 mm, 3 parts

Commit message: generated gerbs
Other:
- board text added: "NO Sensor Breakout"
Changed lines of the file:
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@@
   (general
     (thickness 1.6)
-    (drawings 13)
+    (drawings 15)
     (tracks 15)
     (zones 0)
@@
     (pad_to_mask_clearance 0)
     (aux_axis_origin 0 0)
-    (visible_elements FFFFFF7F)
+    (visible_elements 7FFFFFFF)
     (pcbplotparams
       (layerselection 0x010fc_ffffffff)
@@
       (outputformat 1)
       (mirror false)
-      (drillshape 1)
+      (drillshape 0)
       (scaleselection 1)
-      (outputdirectory ""))
+      (outputdirectory "gerbs/"))
   )
   (net 0 "")
@@
     (tags "mounting hole 2.1mm no annular")
     (attr virtual)
-    (fp_text reference REF** (at 0 -3.2) (layer F.SilkS)
+    (fp_text reference REF** (at 0 -3.2) (layer F.SilkS) hide
       (effects (font (size 1 1) (thickness 0.15)))
     )
@@
       (effects (font (size 1 1) (thickness 0.15)))
     )
+    (fp_circle (center 0 0) (end 2.35 0) (layer F.CrtYd) (width 0.05))
+    (fp_circle (center 0 0) (end 2.1 0) (layer Cmts.User) (width 0.15))
     (fp_text user %R (at 0.3 0) (layer F.Fab)
       (effects (font (size 1 1) (thickness 0.15)))
     )
-    (fp_circle (center 0 0) (end 2.1 0) (layer Cmts.User) (width 0.15))
-    (fp_circle (center 0 0) (end 2.35 0) (layer F.CrtYd) (width 0.05))
     (pad "" np_thru_hole circle (at 0 0) (size 2.1 2.1) (drill 2.1) (layers *.Cu *.Mask))
   )
@@
     (tags "mounting hole 2.1mm no annular")
     (attr virtual)
-    (fp_text reference REF** (at 0 -3.2) (layer F.SilkS)
+    (fp_text reference REF** (at 0 -3.2) (layer F.SilkS) hide
       (effects (font (size 1 1) (thickness 0.15)))
     )
@@
       (effects (font (size 1 1) (thickness 0.15)))
     )
+    (fp_circle (center 0 0) (end 2.35 0) (layer F.CrtYd) (width 0.05))
+    (fp_circle (center 0 0) (end 2.1 0) (layer Cmts.User) (width 0.15))
     (fp_text user %R (at 0.3 0) (layer F.Fab)
       (effects (font (size 1 1) (thickness 0.15)))
     )
-    (fp_circle (center 0 0) (end 2.1 0) (layer Cmts.User) (width 0.15))
-    (fp_circle (center 0 0) (end 2.35 0) (layer F.CrtYd) (width 0.05))
     (pad "" np_thru_hole circle (at 0 0) (size 2.1 2.1) (drill 2.1) (layers *.Cu *.Mask))
   )
@@
       (effects (font (size 1 1) (thickness 0.15)))
     )
+    (fp_line (start -3.175 -13.208) (end 10.795 -13.208) (layer F.SilkS) (width 0.15))
+    (fp_line (start 1.27 -7.62) (end 6.35 -7.62) (layer F.SilkS) (width 0.15))
+    (fp_line (start 5.08 -7.62) (end 5.08 -5.08) (layer F.SilkS) (width 0.15))
+    (fp_line (start 5.08 -5.08) (end 2.54 -5.08) (layer F.SilkS) (width 0.15))
+    (fp_line (start 6.35 -13.208) (end 6.35 -7.62) (layer F.SilkS) (width 0.15))
+    (fp_line (start 10.795 -1.27) (end 10.795 -13.208) (layer F.SilkS) (width 0.15))
+    (fp_line (start 8.89 1.27) (end -1.27 1.27) (layer F.SilkS) (width 0.15))
+    (fp_line (start 1.27 -13.208) (end 1.27 -12.7) (layer F.SilkS) (width 0.15))
+    (fp_line (start -3.175 -1.27) (end -3.175 -13.208) (layer F.SilkS) (width 0.15))
+    (fp_line (start -1.27 -1.27) (end -3.175 -1.27) (layer F.SilkS) (width 0.15))
+    (fp_line (start 1.27 -8.89) (end 1.27 -7.62) (layer F.SilkS) (width 0.15))
+    (fp_line (start 1.27 -8.89) (end 1.27 -12.7) (layer F.SilkS) (width 0.15))
+    (fp_line (start 2.54 -7.62) (end 2.54 -5.08) (layer F.SilkS) (width 0.15))
+    (fp_line (start -1.27 -1.27) (end 10.795 -1.27) (layer F.SilkS) (width 0.15))
+    (fp_line (start 8.89 -1.27) (end 8.89 1.27) (layer F.SilkS) (width 0.15))
     (fp_line (start -1.27 1.27) (end -1.27 -1.27) (layer F.SilkS) (width 0.15))
-    (fp_line (start 8.89 -1.27) (end 8.89 1.27) (layer F.SilkS) (width 0.15))
-    (fp_line (start -1.27 -1.27) (end 10.795 -1.27) (layer F.SilkS) (width 0.15))
-    (fp_line (start 2.54 -7.62) (end 2.54 -5.08) (layer F.SilkS) (width 0.15))
-    (fp_line (start 1.27 -8.89) (end 1.27 -12.7) (layer F.SilkS) (width 0.15))
-    (fp_line (start 1.27 -8.89) (end 1.27 -7.62) (layer F.SilkS) (width 0.15))
-    (fp_line (start -1.27 -1.27) (end -3.175 -1.27) (layer F.SilkS) (width 0.15))
-    (fp_line (start -3.175 -1.27) (end -3.175 -13.208) (layer F.SilkS) (width 0.15))
-    (fp_line (start 1.27 -13.208) (end 1.27 -12.7) (layer F.SilkS) (width 0.15))
-    (fp_line (start 8.89 1.27) (end -1.27 1.27) (layer F.SilkS) (width 0.15))
-    (fp_line (start 10.795 -1.27) (end 10.795 -13.208) (layer F.SilkS) (width 0.15))
-    (fp_line (start 6.35 -13.208) (end 6.35 -7.62) (layer F.SilkS) (width 0.15))
-    (fp_line (start 5.08 -5.08) (end 2.54 -5.08) (layer F.SilkS) (width 0.15))
-    (fp_line (start 5.08 -7.62) (end 5.08 -5.08) (layer F.SilkS) (width 0.15))
-    (fp_line (start 1.27 -7.62) (end 6.35 -7.62) (layer F.SilkS) (width 0.15))
-    (fp_line (start -3.175 -13.208) (end 10.795 -13.208) (layer F.SilkS) (width 0.15))
     (pad 1 thru_hole circle (at 0 0) (size 1.524 1.524) (drill 0.9) (layers *.Cu *.Mask)
       (net 1 +5V))
@@
     )
   )
+  (gr_text "NO Sensor Breakout" (at 137.922 95.25) (layer F.SilkS)
+    (effects (font (size 1.5 1.5) (thickness 0.3)))
+  )
+  (gr_text "NO Sensor Breakout" (at 137.922 95.25) (layer B.SilkS)
+    (effects (font (size 1.5 1.5) (thickness 0.3)) (justify mirror))
+  )
   (gr_line (start 122.936 85.852) (end 124.714 85.852) (layer Edge.Cuts) (width 0.05))
